File: pcb/project/gullwing.kicad_sch (KiCad schematic)
At the start: 7 parts

Commit message: wip
Parts:
- removed C? (x2): 4.7uF, symbol Device:C
- removed C?: 0.1uF, symbol Device:C
- removed L?: DO1608C-103MLB, Inductors:DO1608C, symbol Device:L
- removed U?: TPS62203DBV, Package_TO_SOT_SMD:SOT-23-5, symbol Regulator_Switching:TPS62203DBV
- added C? (x2): C0.1uF, symbol Device:C
- added C? (x2): 4.7uF, symbol Device:C
- added C?: 0.1uF, symbol Device:C
- added L?: DO1608C-103MLB, Inductors:DO1608C, symbol Device:L
- added U?: TPS62203DBV, Package_TO_SOT_SMD:SOT-23-5, symbol Regulator_Switching:TPS62203DBV
Connections:
- net GND: now also C?.1, C?.2, C?.2, C?.2, C?.2, U?.2 (GND); no longer U?.15 (VSS), U?.31 (VSS)
- net USB_DM renamed USB_{DM}
- net USB_DP renamed USB_{DP}
- net V_{cc}_5v renamed V_{cc}
- net V_{cc}: now also C?.1, C?.1, U?.1 (VI), U?.3 (EN)
- net V_{in}_3.3v: no longer names the net of U?.48 (VDD), U?.64 (VDD)
- net V_{in}_3.3v: now also C?.1, C?.1, C?.2, L?.1, U?.4 (FB); no longer U?.16 (VDD), U?.32 (VDD)
- new net: L?.2, U?.5 (SW)
Other:
- moved on the sheet: J?, U?

Commit message: WIP
Parts:
- removed C? (x2): C0.1uF, symbol Device:C
- removed C? (x2): 4.7uF, symbol Device:C
- removed C?: 0.1uF, symbol Device:C
- removed J?: USB_C_Receptacle_USB2.0, symbol Connector:USB_C_Receptacle_USB2.0
- removed L?: DO1608C-103MLB, Inductors:DO1608C, symbol Device:L
- removed U?: TPS62203DBV, Package_TO_SOT_SMD:SOT-23-5, symbol Regulator_Switching:TPS62203DBV
- added C? (x2): 4.7uF, symbol Device:C
- added C? (x5): C0.1uF, symbol Device:C
- added C?: 0.1uF, symbol Device:C
- added J?: USB_C_Receptacle_USB2.0, symbol Connector:USB_C_Receptacle_USB2.0
- added L?: DO1608C-103MLB, Inductors:DO1608C, symbol Device:L
- added U?: TPS62203DBV, Package_TO_SOT_SMD:SOT-23-5, symbol Regulator_Switching:TPS62203DBV
Connections:
- net GND: now also U?.15 (VSS), U?.27 (VSSA), U?.31 (VSS), C?.1, C?.2, C?.2, C?.2, C?.2, C?.2, C?.2, C?.2, J?.A1 (GND), J?.A12 (GND), J?.B1 (GND), J?.B12 (GND), U?.2 (GND)
- net USB_{DM}: now also J?.A7 (D-), J?.B7 (D-)
- net USB_{DP}: now also J?.A6 (D+), J?.B6 (D+)
- net V_{cc}: now also C?.1, C?.1, J?.A4 (VBUS), J?.A9 (VBUS), J?.B4 (VBUS), J?.B9 (VBUS), U?.1 (VI), U?.3 (EN)
- net at U?.48 (VDD), U?.64 (VDD): now also U?.16 (VDD), U?.29 (VDDA), U?.32 (VDD), C?.1, C?.1, C?.1, C?.1, C?.1, C?.2, L?.1, U?.4 (FB)
- new net: L?.2, U?.5 (SW)
Other:
- moved on the sheet: U?
